Commit message: added feedbot descritpion files - this adds the fork to the urdf files

File: niryo_one_description/urdf/v1/niryo_one.urdf.xacro (robot description, xacro)
@@ -27,4 +27,8 @@
     <xacro:property name="distance_wrist_hand_y" value="0" />
     <xacro:property name="distance_hand_tool" value="0.00" />
+    <!-- TSR 2018-19-07 Adding info about test spoon-->
+    <xacro:property name="spoon_offset_x" value="0.14" />
+    <xacro:property name="spoon_offset_y" value="0.0" />
+    <xacro:property name="spoon_offset_z" value="0.067" />
 	<xacro:property name="PI" value="3.14159265359" />
     <xacro:property name="limit_low_shoulder_rotation" value="-3.05433" />
@@ -37,5 +41,5 @@
     <xacro:property name="limit_up_forearm_rotation" value="2.61799" />
     <xacro:property name="limit_low_wrist_rotation" value="-2.26893" />
-    <xacro:property name="limit_up_wrist_rotation" value="2.26893" />
+    <xacro:property name="limit_up_wrist_rotation" value="1.35" />
     <xacro:property name="limit_low_hand_rotation" value="-2.57" />
     <xacro:property name="limit_up_hand_rotation" value="2.57" />
@@ -163,4 +167,6 @@
 	</link>
     <link name="tool_link">
+	</link>
+    <link name="spoon_link">
 	</link>
 	<!--Joints -->
@@ -216,4 +222,9 @@
         <child link="tool_link" />
         <origin xyz="0 0 ${distance_hand_tool}" rpy="${-PI/2} ${-PI/2} 0" />
+    </joint>
+	<joint name="hand_spoon_joint" type="fixed">
+        <parent link="hand_link" />
+        <child link="spoon_link" />
+        <origin xyz="${spoon_offset_x} ${spoon_offset_y} ${spoon_offset_z}" rpy="0 0 0" />
 	</joint>
 </robot>

File: niryo_one_description/urdf/v1/without_mesh_niryo_one.urdf.xacro (robot description, xacro)
@@ -27,4 +27,8 @@
     <xacro:property name="distance_wrist_hand_y" value="0" />
     <xacro:property name="distance_hand_tool" value="0.00" />
+    <!-- TSR 2018-19-07 Adding info about test spoon-->
+    <xacro:property name="spoon_offset_x" value="0.14" />
+    <xacro:property name="spoon_offset_y" value="0.0" />
+    <xacro:property name="spoon_offset_z" value="0.067" />
 	<xacro:property name="PI" value="3.14159265359" />
 	<xacro:property name="limit_low_shoulder_rotation" value="-3.05433" />
@@ -37,5 +41,5 @@
     <xacro:property name="limit_up_forearm_rotation" value="2.61799" />
     <xacro:property name="limit_low_wrist_rotation" value="-2.26893" />
-    <xacro:property name="limit_up_wrist_rotation" value="2.26893" />
+    <xacro:property name="limit_up_wrist_rotation" value="1.35" />
     <xacro:property name="limit_low_hand_rotation" value="-2.57" />
     <xacro:property name="limit_up_hand_rotation" value="2.57" />
@@ -57,4 +61,6 @@
 	</link>
     <link name="tool_link">
+	</link>
+    <link name="spoon_link">
 	</link>
 	<!--Joints -->
@@ -110,4 +116,9 @@
         <child link="tool_link" />
         <origin xyz="0 0 ${distance_hand_tool}" rpy="${-PI/2} ${-PI/2} 0" />
+    </joint>
+	<joint name="hand_spoon_joint" type="fixed">
+        <parent link="hand_link" />
+        <child link="spoon_link" />
+        <origin xyz="${spoon_offset_x} ${spoon_offset_y} ${spoon_offset_z}" rpy="0 0 0" />
 	</joint>
 </robot>

File: niryo_one_description/urdf/v2/niryo_one.urdf.xacro (robot description, xacro)
@@ -16,4 +16,6 @@
 -->
 <robot xmlns:xacro="http://www.ros.org/wiki/xacro" name="niryo_one">
+        <!-- Add an xacro arg to simulate tf_prefix -->
+    <xacro:arg name="link_prefix" default=""/>
 	<!-- Properties -->
     <xacro:property name="distance_origin_shoulder_z" value="0.103" />
@@ -27,4 +29,10 @@
     <xacro:property name="distance_wrist_hand_y" value="-0.0055" />
     <xacro:property name="distance_hand_tool" value="0.0073" />
+        <!-- TSR 2018-19-07 Adding info about test spoon-->
+    <xacro:property name="spoon_offset_x" value="0.14" />
+    <xacro:property name="spoon_offset_y" value="0.0" />
+    <xacro:property name="spoon_offset_z" value="0.067" />
+    <xacro:property name="thickness_arm_axis" value="0.052" />
+    <xacro:property name="thickness_forearm_axis" value="0.048" />
 	<xacro:property name="PI" value="3.14159265359" />
     <xacro:property name="limit_low_shoulder_rotation" value="-3.05433" />
@@ -41,6 +49,6 @@
     <xacro:property name="limit_up_hand_rotation" value="2.57436" />
 	<!-- Links -->
-    <link name="ground_link"/>
-    <link name="base_link">
+    <link name="$(arg link_prefix)ground_link"/>
+    <link name="$(arg link_prefix)base_link">
 		<visual>
 			<origin xyz="0 0 0" rpy="0 0 0" />
@@ -56,5 +64,5 @@
         </collision>
 	</link>
-    <link name="shoulder_link">
+    <link name="$(arg link_prefix)shoulder_link">
 		<visual>
 			<origin xyz="0 0 0" rpy="0 0 0" />
@@ -70,5 +78,5 @@
         </collision>
 	</link>
-    <link name="arm_link">
+    <link name="$(arg link_prefix)arm_link">
 		<visual>
 			<origin xyz="0 0 0" rpy="0 0 0" />
@@ -84,5 +92,5 @@
         </collision>
 	</link>
-    <link name="elbow_link">
+    <link name="$(arg link_prefix)elbow_link">
 		<visual>
 			<origin xyz="0 0 0" rpy="0 0 0" />
@@ -98,5 +106,5 @@
         </collision>
 	</link>
-    <link name="forearm_link">
+    <link name="$(arg link_prefix)forearm_link">
 		<visual>
 			<origin xyz="0 0 0" rpy="0 0 0" />
@@ -112,5 +120,5 @@
         </collision>
 	</link>
-    <link name="wrist_link">
+    <link name="$(arg link_prefix)wrist_link">
 		<visual>
 			<origin xyz="0 0 0" rpy="0 0 0" />
@@ -126,5 +134,5 @@
         </collision>
 	</link>
-    <link name="hand_link">
+    <link name="$(arg link_prefix)hand_link">
 		<visual>
 			<origin xyz="0 0 0" rpy="0 0 0" />
@@ -140,15 +148,17 @@
         </collision>
 	</link>
-    <link name="tool_link">
+    <link name="$(arg link_prefix)tool_link">
+	</link>
+    <link name="$(arg link_prefix)spoon_link">
 	</link>
 	<!--Joints -->
     <joint name="ground_joint" type="fixed">
-        <parent link="ground_link" />
-        <child link="base_link" />
+        <parent link="$(arg link_prefix)ground_link" />
+        <child link="$(arg link_prefix)base_link" />
         <origin xyz="0 0 0" rpy="0 0 0" />
     </joint>
 	<joint name="joint_1" type="revolute">
-        <parent link="base_link" />
-        <child link="shoulder_link" />
+        <parent link="$(arg link_prefix)base_link" />
+        <child link="$(arg link_prefix)shoulder_link" />
 		<origin xyz="0 0 ${distance_origin_shoulder_z}" rpy="0 0 0" />
 		<axis xyz="0 0 1" />
@@ -156,6 +166,6 @@
 	</joint>
 	<joint name="joint_2" type="revolute">
-        <parent link="shoulder_link" />
-        <child link="arm_link" />
+        <parent link="$(arg link_prefix)shoulder_link" />
+        <child link="$(arg link_prefix)arm_link" />
         <origin xyz="0 0 ${distance_shoulder_arm_z}" rpy="${PI/2} ${-PI/2} 0" />
 		<limit effort="1" velocity="1.0" lower="${limit_low_arm_rotation}" upper="${limit_up_arm_rotation}" />
@@ -163,6 +173,6 @@
 	</joint>
 	<joint name="joint_3" type="revolute">
-        <parent link="arm_link" />
-        <child link="elbow_link" />
+        <parent link="$(arg link_prefix)arm_link" />
+        <child link="$(arg link_prefix)elbow_link" />
         <origin xyz="${distance_arm_elbow_x} ${distance_arm_elbow_y} 0" rpy="0 0 ${-PI/2}" />
 		<limit effort="1" velocity="1.0" lower="${limit_low_elbow_rotation}" upper="${limit_up_elbow_rotation}" />
@@ -170,6 +180,6 @@
 	</joint>
 	<joint name="joint_4" type="revolute">
-        <parent link="elbow_link" />
-        <child link="forearm_link" />
+        <parent link="$(arg link_prefix)elbow_link" />
+        <child link="$(arg link_prefix)forearm_link" />
         <origin xyz="${distance_elbow_forearm_x} ${distance_elbow_forearm_y} 0" rpy="0 ${PI/2} 0" />
 		<limit effort="1" velocity="1.0" lower="${limit_low_forearm_rotation}" upper="${limit_up_forearm_rotation}" />
@@ -177,6 +187,6 @@
 	</joint>
 	<joint name="joint_5" type="revolute">
-        <parent link="forearm_link" />
-        <child link="wrist_link" />
+        <parent link="$(arg link_prefix)forearm_link" />
+        <child link="$(arg link_prefix)wrist_link" />
 		<origin xyz="0 0 ${distance_forearm_wrist_z}" rpy="0 ${-PI/2} 0" />
 		<limit effort="1" velocity="1.0" lower="${limit_low_wrist_rotation}" upper="${limit_up_wrist_rotation}" />
@@ -184,6 +194,6 @@
 	</joint>
 	<joint name="joint_6" type="revolute">
-        <parent link="wrist_link" />
-        <child link="hand_link" />
+        <parent link="$(arg link_prefix)wrist_link" />
+        <child link="$(arg link_prefix)hand_link" />
         <origin xyz="${distance_wrist_hand_x} ${distance_wrist_hand_y} 0" rpy="0 ${PI/2} 0" />
 		<limit effort="1" velocity="1.0" lower="${limit_low_hand_rotation}" upper="${limit_up_hand_rotation}" />
@@ -191,7 +201,12 @@
 	</joint>
 	<joint name="hand_tool_joint" type="fixed">
-        <parent link="hand_link" />
-        <child link="tool_link" />
+        <parent link="$(arg link_prefix)hand_link" />
+        <child link="$(arg link_prefix)tool_link" />
         <origin xyz="0 0 ${distance_hand_tool}" rpy="${-PI/2} ${-PI/2} 0" />
+    </joint>
+	<joint name="hand_spoon_joint" type="fixed">
+        <parent link="$(arg link_prefix)hand_link" />
+        <child link="$(arg link_prefix)spoon_link" />
+        <origin xyz="${spoon_offset_x} ${spoon_offset_y} ${spoon_offset_z}" rpy="0 0 0" />
 	</joint>
 </robot>

File: niryo_one_description/urdf/v2/without_mesh_niryo_one.urdf.xacro (robot description, xacro)
@@ -27,4 +27,8 @@
     <xacro:property name="distance_wrist_hand_y" value="-0.0055" />
     <xacro:property name="distance_hand_tool" value="0.0073" />
+	    <!-- TSR 2018-19-07 Adding info about test spoon-->
+    <xacro:property name="spoon_offset_x" value="0.14" />
+    <xacro:property name="spoon_offset_y" value="0.0" />
+    <xacro:property name="spoon_offset_z" value="0.067" />
 	<xacro:property name="PI" value="3.14159265359" />
     <xacro:property name="limit_low_shoulder_rotation" value="-3.05433" />
@@ -57,4 +61,6 @@
 	</link>
     <link name="tool_link">
+	</link>
+    <link name="spoon_link">
 	</link>
 	<!--Joints -->
@@ -111,3 +117,8 @@
         <origin xyz="0 0 ${distance_hand_tool}" rpy="${-PI/2} ${-PI/2} 0" />
 	</joint>
+    <joint name="hand_spoon_joint" type="fixed">
+        <parent link="hand_link" />
+        <child link="spoon_link" />
+        <origin xyz="${spoon_offset_x} ${spoon_offset_y} ${spoon_offset_z}" rpy="0 0 0" />
+	</joint>
 </robot>

Commit message: changed the spoon size to 17cm

File: niryo_one_description/urdf/v1/niryo_one.urdf.xacro (robot description, xacro)
@@ -28,5 +28,5 @@
     <xacro:property name="distance_hand_tool" value="0.00" />
     <!-- TSR 2018-19-07 Adding info about test spoon-->
-    <xacro:property name="spoon_offset_x" value="0.14" />
+    <xacro:property name="spoon_offset_x" value="0.17" />
     <xacro:property name="spoon_offset_y" value="0.0" />
     <xacro:property name="spoon_offset_z" value="0.067" />

File: niryo_one_description/urdf/v1/without_mesh_niryo_one.urdf.xacro (robot description, xacro)
@@ -28,5 +28,5 @@
     <xacro:property name="distance_hand_tool" value="0.00" />
     <!-- TSR 2018-19-07 Adding info about test spoon-->
-    <xacro:property name="spoon_offset_x" value="0.14" />
+    <xacro:property name="spoon_offset_x" value="0.17" />
     <xacro:property name="spoon_offset_y" value="0.0" />
     <xacro:property name="spoon_offset_z" value="0.067" />

File: niryo_one_description/urdf/v2/niryo_one.urdf.xacro (robot description, xacro)
@@ -30,5 +30,5 @@
     <xacro:property name="distance_hand_tool" value="0.0073" />
         <!-- TSR 2018-19-07 Adding info about test spoon-->
-    <xacro:property name="spoon_offset_x" value="0.14" />
+    <xacro:property name="spoon_offset_x" value="0.17" />
     <xacro:property name="spoon_offset_y" value="0.0" />
     <xacro:property name="spoon_offset_z" value="0.067" />

File: niryo_one_description/urdf/v2/without_mesh_niryo_one.urdf.xacro (robot description, xacro)
@@ -28,5 +28,5 @@
     <xacro:property name="distance_hand_tool" value="0.0073" />
 	    <!-- TSR 2018-19-07 Adding info about test spoon-->
-    <xacro:property name="spoon_offset_x" value="0.14" />
+    <xacro:property name="spoon_offset_x" value="0.17" />
     <xacro:property name="spoon_offset_y" value="0.0" />
     <xacro:property name="spoon_offset_z" value="0.067" />

Commit message: changed the description of the robot to new end-effector

File: niryo_one_description/urdf/v1/niryo_one.urdf.xacro (robot description, xacro)
@@ -28,7 +28,7 @@
     <xacro:property name="distance_hand_tool" value="0.00" />
     <!-- TSR 2018-19-07 Adding info about test spoon-->
-    <xacro:property name="spoon_offset_x" value="0.17" />
+    <xacro:property name="spoon_offset_x" value="0.16" />
     <xacro:property name="spoon_offset_y" value="0.0" />
-    <xacro:property name="spoon_offset_z" value="0.067" />
+    <xacro:property name="spoon_offset_z" value="0.065" />
 	<xacro:property name="PI" value="3.14159265359" />
     <xacro:property name="limit_low_shoulder_rotation" value="-3.05433" />

File: niryo_one_description/urdf/v1/without_mesh_niryo_one.urdf.xacro (robot description, xacro)
@@ -28,7 +28,7 @@
     <xacro:property name="distance_hand_tool" value="0.00" />
     <!-- TSR 2018-19-07 Adding info about test spoon-->
-    <xacro:property name="spoon_offset_x" value="0.17" />
+    <xacro:property name="spoon_offset_x" value="0.16" />
     <xacro:property name="spoon_offset_y" value="0.0" />
-    <xacro:property name="spoon_offset_z" value="0.067" />
+    <xacro:property name="spoon_offset_z" value="0.065" />
 	<xacro:property name="PI" value="3.14159265359" />
 	<xacro:property name="limit_low_shoulder_rotation" value="-3.05433" />

File: niryo_one_description/urdf/v2/niryo_one.urdf.xacro (robot description, xacro)
@@ -30,7 +30,7 @@
     <xacro:property name="distance_hand_tool" value="0.0073" />
         <!-- TSR 2018-19-07 Adding info about test spoon-->
-    <xacro:property name="spoon_offset_x" value="0.17" />
+    <xacro:property name="spoon_offset_x" value="0.16" />
     <xacro:property name="spoon_offset_y" value="0.0" />
-    <xacro:property name="spoon_offset_z" value="0.067" />
+    <xacro:property name="spoon_offset_z" value="0.065" />
     <xacro:property name="thickness_arm_axis" value="0.052" />
     <xacro:property name="thickness_forearm_axis" value="0.048" />

File: niryo_one_description/urdf/v2/without_mesh_niryo_one.urdf.xacro (robot description, xacro)
@@ -28,7 +28,7 @@
     <xacro:property name="distance_hand_tool" value="0.0073" />
 	    <!-- TSR 2018-19-07 Adding info about test spoon-->
-    <xacro:property name="spoon_offset_x" value="0.17" />
+    <xacro:property name="spoon_offset_x" value="0.16" />
     <xacro:property name="spoon_offset_y" value="0.0" />
-    <xacro:property name="spoon_offset_z" value="0.067" />
+    <xacro:property name="spoon_offset_z" value="0.065" />
 	<xacro:property name="PI" value="3.14159265359" />
     <xacro:property name="limit_low_shoulder_rotation" value="-3.05433" />
