Commit message: almost there - depth image ok

File: feedbot_gazebo/models/realsense_camera/urdf/_d415.urdf.xacro (robot description, xacro)
@@ -46,5 +46,5 @@
         <geometry>
           <!-- <box size="${d415_cam_width} ${d415_cam_height} ${d415_cam_depth}"/> -->
-          <mesh filename="package://feedbot_description/meshes/camera/stl/d415.stl" />
+          <mesh filename="package://feedbot_gazebo/models/realsense_camera/meshes/d415.dae" />
         </geometry>
         <material name="aluminum"/>
