Commit message: simulation ok - still need to find if depth camera is ok or not

File: feedbot_gazebo/models/realsense_camera/urdf/feedbot_camera.urdf.xacro (robot description, xacro)
@@ -6,10 +6,9 @@
     xmlns:xacro="http://playerstage.sourceforge.net/gazebo/xmlschema/#xacro">
     <xacro:include filename="$(find feedbot_gazebo)/models/realsense_camera/urdf/_d415.urdf.xacro" />
-    <link name="feedbot_camera_base_link"/>
+    <link name="feedbot_camera_base_link"></link>
     <sensor_d415 parent="feedbot_camera_base_link">
        <origin xyz="0 0 0" rpy="0 0 0"/>
     </sensor_d415>
     <gazebo reference="feedbot_camera_base_link">
-        <gravity>0</gravity>
         <sensor name="color" type="camera">
             <pose frame="camera_color_optical_frame">0 0 0 0 0 0</pose>
