Commit message: added package with feedbot specific description and bringup

File: feedbot_description/urdf/feedbot_v2_wmesh.urdf.xacro (robot description, xacro)
@@ -214,11 +214,11 @@
 			<origin xyz="0 0 0" rpy="0 0 0" />
 			<geometry>
-                <mesh filename="package://niryo_one_description/meshes/feedbot_parts/collada/spoon_holder.dae" />
-			</geometry>
-		</visual>
-        <collision>
-			<origin xyz="0 0 0" rpy="0 0 0" />
-            <geometry>
-                <mesh filename="package://niryo_one_description/meshes/feedbot_parts/stl/spoon_holder.stl" />
+                <mesh filename="package://feedbot_description/meshes/feedbot_parts/collada/spoon_holder.dae" />
+			</geometry>
+		</visual>
+        <collision>
+			<origin xyz="0 0 0" rpy="0 0 0" />
+            <geometry>
+                <mesh filename="package://feedbot_description/meshes/feedbot_parts/stl/spoon_holder.stl" />
             </geometry>
         </collision>

Commit message: added spoon to spoon holder model, and changed the tip of the spoon location

File: feedbot_description/urdf/feedbot_v2_wmesh.urdf.xacro (robot description, xacro)
@@ -30,7 +30,7 @@
     <xacro:property name="distance_hand_tool" value="0.0073" />
         <!-- TSR 2018-19-07 Adding info about test spoon-->
-    <xacro:property name="spoon_offset_x" value="0.16" />
-    <xacro:property name="spoon_offset_y" value="0.0" />
-    <xacro:property name="spoon_offset_z" value="0.065" />
+    <xacro:property name="spoon_offset_x" value="0.060" />
+    <xacro:property name="spoon_offset_y" value="0.171" />
+    <xacro:property name="spoon_offset_z" value="-0.016" />
     <xacro:property name="thickness_arm_axis" value="0.052" />
     <xacro:property name="thickness_forearm_axis" value="0.048" />
@@ -292,6 +292,6 @@
         <origin xyz="0 0 0" rpy="0 0 0" />
 	</joint>
-	<joint name="hand_spoon_joint" type="fixed">
-        <parent link="$(arg link_prefix)hand_link" />
+	<joint name="spoon_joint" type="fixed">
+        <parent link="$(arg link_prefix)spoon_holder_link" />
         <child link="$(arg link_prefix)spoon_link" />
         <origin xyz="${spoon_offset_x} ${spoon_offset_y} ${spoon_offset_z}" rpy="0 0 0" />

Commit message: vizualization working in rviz and moveit planning working in ros-melodic

File: feedbot_description/urdf/feedbot_v2_wmesh.urdf.xacro (robot description, xacro)
@@ -1,3 +1,7 @@
-<?xml version="1.0"?>
+<?xml version="1.0" encoding="utf-8" ?>
+<!-- =================================================================================== -->
+<!-- |    This document was autogenerated by xacro from /home/acandeias/ROSws/feedbot_ws/src/niryo_one_ros/feedbot_description/urdf/feedbot_v2_wmesh.urdf.xacro | -->
+<!-- |    EDITING THIS FILE BY HAND IS NOT RECOMMENDED                                 | -->
+<!-- =================================================================================== -->
 <!--
     niryo_one.urdf.xacro
@@ -15,51 +19,102 @@
     along with this program.  If not, see <http://www.gnu.org/licenses/>.
 -->
-<robot xmlns:xacro="http://www.ros.org/wiki/xacro" name="niryo_one">
-        <!-- Add an xacro arg to simulate tf_prefix -->
-    <xacro:arg name="link_prefix" default=""/>
-	<!-- Properties -->
-    <xacro:property name="distance_origin_shoulder_z" value="0.103" />
-    <xacro:property name="distance_shoulder_arm_z" value="0.080" />
-    <xacro:property name="distance_arm_elbow_x" value="0.210" />
-    <xacro:property name="distance_arm_elbow_y" value="0.0" />
-    <xacro:property name="distance_elbow_forearm_x" value="0.0415" />
-    <xacro:property name="distance_elbow_forearm_y" value="0.030" />
-    <xacro:property name="distance_forearm_wrist_z" value="0.180" />
-    <xacro:property name="distance_wrist_hand_x" value="0.0164" />
-    <xacro:property name="distance_wrist_hand_y" value="-0.0055" />
-    <xacro:property name="distance_hand_tool" value="0.0073" />
-        <!-- TSR 2018-19-07 Adding info about test spoon-->
-    <xacro:property name="spoon_offset_x" value="0.060" />
-    <xacro:property name="spoon_offset_y" value="0.171" />
-    <xacro:property name="spoon_offset_z" value="-0.016" />
-    <xacro:property name="thickness_arm_axis" value="0.052" />
-    <xacro:property name="thickness_forearm_axis" value="0.048" />
-	<xacro:property name="PI" value="3.14159265359" />
-    <xacro:property name="limit_low_shoulder_rotation" value="-3.05433" />
-    <xacro:property name="limit_up_shoulder_rotation" value="3.05433" />
-    <xacro:property name="limit_low_arm_rotation" value="-1.91986" />
-    <xacro:property name="limit_up_arm_rotation" value="0.640187" />
-    <xacro:property name="limit_low_elbow_rotation" value="-1.397485" />
-    <xacro:property name="limit_up_elbow_rotation" value="${PI/2}" />
-    <xacro:property name="limit_low_forearm_rotation" value="-3.05433" />
-    <xacro:property name="limit_up_forearm_rotation" value="3.05433" />
-    <xacro:property name="limit_low_wrist_rotation" value="-1.74533" />
-    <xacro:property name="limit_up_wrist_rotation" value="1.91986" />
-    <xacro:property name="limit_low_hand_rotation" value="-2.57436" />
-    <xacro:property name="limit_up_hand_rotation" value="2.57436" />
-    <xacro:include filename="$(find niryo_one_description)/urdf/gazebo/niryo_one_v2.gazebo.xacro" />
-	<xacro:include filename="$(find niryo_one_description)/urdf/gazebo/utils.xacro" />
-	<xacro:include filename="$(find niryo_one_description)/urdf/gazebo/niryo_one.transmission.xacro" />
-	<!-- Links -->
-    <link name="$(arg link_prefix)ground_link"/>
-    <link name="$(arg link_prefix)base_link">
-		<visual>
-			<origin xyz="0 0 0" rpy="0 0 0" />
-			<geometry>
+<robot name="niryo_one" xmlns:xacro="http://www.ros.org/wiki/xacro">
+    <!-- Properties -->
+    <gazebo reference="ground_link">
+        <turnGravityOff>true</turnGravityOff>
+    </gazebo>
+    <gazebo reference="base_link">
+        <turnGravityOff>true</turnGravityOff>
+    </gazebo>
+    <gazebo reference="shoulder_link">
+        <turnGravityOff>true</turnGravityOff>
+    </gazebo>
+    <gazebo reference="arm_link">
+        <turnGravityOff>true</turnGravityOff>
+    </gazebo>
+    <gazebo reference="elbow_link">
+        <turnGravityOff>true</turnGravityOff>
+    </gazebo>
+    <gazebo reference="forearm_link">
+        <turnGravityOff>true</turnGravityOff>
+    </gazebo>
+    <gazebo reference="wrist_link">
+        <turnGravityOff>true</turnGravityOff>
+    </gazebo>
+    <gazebo reference="hand_link">
+        <turnGravityOff>true</turnGravityOff>
+    </gazebo>
+    <gazebo reference="tool_link">
+        <turnGravityOff>true</turnGravityOff>
+    </gazebo>
+    <!--transmission-->
+    <transmission name="base_shoulder_transmission">
+        <type>transmission_interface/SimpleTransmission</type>
+        <joint name="joint_1">
+            <hardwareInterface>hardware_interface/PositionJointInterface</hardwareInterface>
+        </joint>
+        <actuator name="base_shoulder_stepper">
+            <mechanicalReduction>6.0625</mechanicalReduction>
+            <hardwareInterface>hardware_interface/PositionJointInterface</hardwareInterface>
+        </actuator>
+    </transmission>
+    <transmission name="shoulder_arm_transmission">
+        <type>transmission_interface/SimpleTransmission</type>
+        <joint name="joint_2">
+            <hardwareInterface>hardware_interface/PositionJointInterface</hardwareInterface>
+        </joint>
+        <actuator name="shoulder_arm_stepper">
+            <mechanicalReduction>8.3125</mechanicalReduction>
+            <hardwareInterface>hardware_interface/PositionJointInterface</hardwareInterface>
+        </actuator>
+    </transmission>
+    <transmission name="arm_elbow_transmission">
+        <type>transmission_interface/SimpleTransmission</type>
+        <joint name="joint_3">
+            <hardwareInterface>hardware_interface/PositionJointInterface</hardwareInterface>
+        </joint>
+        <actuator name="arm_elbow_stepper">
+            <mechanicalReduction>7.875</mechanicalReduction>
+            <hardwareInterface>hardware_interface/PositionJointInterface</hardwareInterface>
+        </actuator>
+    </transmission>
+    <transmission name="elbow_forarm_transmission">
+        <type>transmission_interface/SimpleTransmission</type>
+        <joint name="joint_4">
+            <hardwareInterface>hardware_interface/PositionJointInterface</hardwareInterface>
+        </joint>
+        <actuator name="elbow_forarm_motor">
+            <mechanicalReduction>5.0</mechanicalReduction>
+        </actuator>
+    </transmission>
+    <transmission name="forarm_wirst_transmission">
+        <type>transmission_interface/SimpleTransmission</type>
+        <joint name="joint_5">
+            <hardwareInterface>hardware_interface/PositionJointInterface</hardwareInterface>
+        </joint>
+        <actuator name="forarm_wirst_motor">
+            <mechanicalReduction>1</mechanicalReduction>
+        </actuator>
+    </transmission>
+    <transmission name="wirst_gripper_transmission">
+        <type>transmission_interface/SimpleTransmission</type>
+        <joint name="joint_6">
+            <hardwareInterface>hardware_interface/PositionJointInterface</hardwareInterface>
+        </joint>
+        <actuator name="wirst_gripper_motor">
+            <mechanicalReduction>1</mechanicalReduction>
+        </actuator>
+    </transmission>
+    <!-- Links -->
+    <link name="ground_link" />
+    <link name="base_link">
+        <visual>
+            <origin rpy="0 0 0" xyz="0 0 0" />
+            <geometry>
                 <mesh filename="package://niryo_one_description/meshes/v2/collada/base_link.dae" />
-			</geometry>
-        </visual>
-        <collision>
-			<origin xyz="0 0 0" rpy="0 0 0" />
+            </geometry>
+        </visual>
+        <collision>
+            <origin rpy="0 0 0" xyz="0 0 0" />
             <geometry>
                 <mesh filename="package://niryo_one_description/meshes/v2/stl/base_link.stl" />
@@ -67,22 +122,19 @@
         </collision>
         <inertial>
-      		<origin xyz="0 0 0" rpy="0 0 0"/>
-      		<mass value="2"/>
-			<!--to change-->
-      		<inertia
-        		ixx="0.0" ixy="0.0" ixz="0.0"
-        		iyy="0.0" iyz="0.0"
-        		izz="0.0"/>
-    	</inertial>
-	</link>
-    <link name="$(arg link_prefix)shoulder_link">
-		<visual>
-			<origin xyz="0 0 0" rpy="0 0 0" />
-			<geometry>
+            <origin rpy="0 0 0" xyz="0 0 0" />
+            <mass value="2" />
+            <!--to change-->
+            <inertia ixx="0.0" ixy="0.0" ixz="0.0" iyy="0.0" iyz="0.0" izz="0.0" />
+        </inertial>
+    </link>
+    <link name="shoulder_link">
+        <visual>
+            <origin rpy="0 0 0" xyz="0 0 0" />
+            <geometry>
                 <mesh filename="package://niryo_one_description/meshes/v2/collada/shoulder_link.dae" />
-			</geometry>
-		</visual>
-        <collision>
-			<origin xyz="0 0 0" rpy="0 0 0" />
+            </geometry>
+        </visual>
+        <collision>
+            <origin rpy="0 0 0" xyz="0 0 0" />
             <geometry>
                 <mesh filename="package://niryo_one_description/meshes/v2/stl/shoulder_link.stl" />
@@ -90,21 +142,18 @@
         </collision>
         <inertial>
-      		<origin xyz="0 0 0" rpy="0 0 0"/>
-      		<mass value="1"/>
-      		<inertia
-        		ixx="1.0" ixy="0.0" ixz="0.0"
-        		iyy="1.0" iyz="0.0"
-        		izz="1.0"/>
-    	</inertial>
-	</link>
-    <link name="$(arg link_prefix)arm_link">
-		<visual>
-			<origin xyz="0 0 0" rpy="0 0 0" />
-			<geometry>
+            <origin rpy="0 0 0" xyz="0 0 0" />
+            <mass value="1" />
+            <inertia ixx="1.0" ixy="0.0" ixz="0.0" iyy="1.0" iyz="0.0" izz="1.0" />
+        </inertial>
+    </link>
+    <link name="arm_link">
+        <visual>
+            <origin rpy="0 0 0" xyz="0 0 0" />
+            <geometry>
                 <mesh filename="package://niryo_one_description/meshes/v2/collada/arm_link.dae" />
-			</geometry>
-		</visual>
-        <collision>
-			<origin xyz="0 0 0" rpy="0 0 0" />
+            </geometry>
+        </visual>
+        <collision>
+            <origin rpy="0 0 0" xyz="0 0 0" />
             <geometry>
                 <mesh filename="package://niryo_one_description/meshes/v2/stl/arm_link.stl" />
@@ -112,21 +161,18 @@
         </collision>
         <inertial>
-      		<origin xyz="0 0 0" rpy="0 0 0"/>
-      		<mass value="0.5"/>
-      		<inertia
-        		ixx="1.0" ixy="0.0" ixz="0.0"
-        		iyy="1.0" iyz="0.0"
-        		izz="1.0"/>
-    	</inertial>
-	</link>
-    <link name="$(arg link_prefix)elbow_link">
-		<visual>
-			<origin xyz="0 0 0" rpy="0 0 0" />
-			<geometry>
+            <origin rpy="0 0 0" xyz="0 0 0" />
+            <mass value="0.5" />
+            <inertia ixx="1.0" ixy="0.0" ixz="0.0" iyy="1.0" iyz="0.0" izz="1.0" />
+        </inertial>
+    </link>
+    <link name="elbow_link">
+        <visual>
+            <origin rpy="0 0 0" xyz="0 0 0" />
+            <geometry>
                 <mesh filename="package://niryo_one_description/meshes/v2/collada/elbow_link.dae" />
-			</geometry>
-		</visual>
-        <collision>
-			<origin xyz="0 0 0" rpy="0 0 0" />
+            </geometry>
+        </visual>
+        <collision>
+            <origin rpy="0 0 0" xyz="0 0 0" />
             <geometry>
                 <mesh filename="package://niryo_one_description/meshes/v2/stl/elbow_link.stl" />
@@ -134,21 +180,18 @@
         </collision>
         <inertial>
-      		<origin xyz="0 0 0" rpy="0 0 0"/>
-      		<mass value="0.4"/>
-      		<inertia
-        		ixx="1.0" ixy="0.0" ixz="0.0"
-        		iyy="1.0" iyz="0.0"
-        		izz="1.0"/>
-    	</inertial>
-	</link>
-    <link name="$(arg link_prefix)forearm_link">
-		<visual>
-			<origin xyz="0 0 0" rpy="0 0 0" />
-			<geometry>
+            <origin rpy="0 0 0" xyz="0 0 0" />
+            <mass value="0.4" />
+            <inertia ixx="1.0" ixy="0.0" ixz="0.0" iyy="1.0" iyz="0.0" izz="1.0" />
+        </inertial>
+    </link>
+    <link name="forearm_link">
+        <visual>
+            <origin rpy="0 0 0" xyz="0 0 0" />
+            <geometry>
                 <mesh filename="package://niryo_one_description/meshes/v2/collada/forearm_link.dae" />
-			</geometry>
-		</visual>
-        <collision>
-			<origin xyz="0 0 0" rpy="0 0 0" />
+            </geometry>
+        </visual>
+        <collision>
+            <origin rpy="0 0 0" xyz="0 0 0" />
             <geometry>
                 <mesh filename="package://niryo_one_description/meshes/v2/stl/forearm_link.stl" />
@@ -156,21 +199,18 @@
         </collision>
         <inertial>
-      		<origin xyz="0 0 0" rpy="0 0 0"/>
-      		<mass value="0.3"/>
-      		<inertia
-        		ixx="1.0" ixy="0.0" ixz="0.0"
-        		iyy="1.0" iyz="0.0"
-        		izz="1.0"/>
-    	</inertial>
-	</link>
-    <link name="$(arg link_prefix)wrist_link">
-		<visual>
-			<origin xyz="0 0 0" rpy="0 0 0" />
-			<geometry>
+            <origin rpy="0 0 0" xyz="0 0 0" />
+            <mass value="0.3" />
+            <inertia ixx="1.0" ixy="0.0" ixz="0.0" iyy="1.0" iyz="0.0" izz="1.0" />
+        </inertial>
+    </link>
+    <link name="wrist_link">
+        <visual>
+            <origin rpy="0 0 0" xyz="0 0 0" />
+            <geometry>
                 <mesh filename="package://niryo_one_description/meshes/v2/collada/wrist_link.dae" />
-			</geometry>
-		</visual>
-        <collision>
-			<origin xyz="0 0 0" rpy="0 0 0" />
+            </geometry>
+        </visual>
+        <collision>
+            <origin rpy="0 0 0" xyz="0 0 0" />
             <geometry>
                 <mesh filename="package://niryo_one_description/meshes/v2/stl/wrist_link.stl" />
@@ -178,21 +218,18 @@
         </collision>
         <inertial>
-      		<origin xyz="0 0 0" rpy="0 0 0"/>
-      		<mass value="0.2"/>
-      		<inertia
-        		ixx="1.0" ixy="0.0" ixz="0.0"
-        		iyy="1.0" iyz="0.0"
-        		izz="1.0"/>
-    	</inertial>
-	</link>
-    <link name="$(arg link_prefix)hand_link">
-		<visual>
-			<origin xyz="0 0 0" rpy="0 0 0" />
-			<geometry>
+            <origin rpy="0 0 0" xyz="0 0 0" />
+            <mass value="0.2" />
+            <inertia ixx="1.0" ixy="0.0" ixz="0.0" iyy="1.0" iyz="0.0" izz="1.0" />
+        </inertial>
+    </link>
+    <link name="hand_link">
+        <visual>
+            <origin rpy="0 0 0" xyz="0 0 0" />
+            <geometry>
                 <mesh filename="package://niryo_one_description/meshes/v2/collada/hand_link.dae" />
-			</geometry>
-		</visual>
-        <collision>
-			<origin xyz="0 0 0" rpy="0 0 0" />
+            </geometry>
+        </visual>
+        <collision>
+            <origin rpy="0 0 0" xyz="0 0 0" />
             <geometry>
                 <mesh filename="package://niryo_one_description/meshes/v2/stl/hand_link.stl" />
@@ -200,104 +237,160 @@
         </collision>
         <inertial>
-      		<origin xyz="0 0 0" rpy="0 0 0"/>
-      		<mass value="0.1"/>
-      		<inertia
-        		ixx="1.0" ixy="0.0" ixz="0.0"
-        		iyy="1.0" iyz="0.0"
-        		izz="1.0"/>
-    	</inertial>
-	</link>
-    <link name="$(arg link_prefix)tool_link">
-	</link>
-	<link name="$(arg link_prefix)spoon_holder_link">
-		<visual>
-			<origin xyz="0 0 0" rpy="0 0 0" />
-			<geometry>
+            <origin rpy="0 0 0" xyz="0 0 0" />
+            <mass value="0.1" />
+            <inertia ixx="1.0" ixy="0.0" ixz="0.0" iyy="1.0" iyz="0.0" izz="1.0" />
+        </inertial>
+    </link>
+    <link name="tool_link" />
+    <link name="spoon_holder_link">
+        <visual>
+            <origin rpy="0 0 0" xyz="0 0 0" />
+            <geometry>
                 <mesh filename="package://feedbot_description/meshes/feedbot_parts/collada/spoon_holder.dae" />
-			</geometry>
-		</visual>
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